Commit message: 2/11/18

File: src/two_wheels_description/urdf/2wheels_with_arm.urdf (robot description, URDF)
Before this commit: robot 2wheels, 13 links, 12 joints
Links:
- removed link link_chassis
- added link base_link, mass 10.0; collision box size=0.18 0.2 0.06; visual mesh filename=package://two_wheels_description/meshes/robotmodel.dae
Joints:
- joint camera_joint: origin xyz=0.0 0.11 0.02 rpy=0 0 1.5708 -> xyz=0.11 0.0 0.02 rpy=0 0 0; parent link_chassis -> base_link
- joint joint_caster: limit effort=1000 velocity=100 -> effort=1000 velocity=10; origin xyz=0.008 0.085 -0.015 rpy=0 0 0 -> xyz=0.085 -0.008 -0.015 rpy=0 0 0; parent link_chassis -> base_link
- joint joint_left_wheel: axis 0 0 1 -> 0 0 -1; origin xyz=-0.11 -0.057 0.012 rpy=0 -1.570 0 -> xyz=-0.0572 0.11  0.012 rpy=1.5707 0  0; parent link_chassis -> base_link
- joint joint_right_wheel: axis 0 0 -1 -> 0 0 1; origin xyz=0.11 -0.057 0.012 rpy=0 1.570 0 -> xyz=-0.0572 -0.11 0.012 rpy=-1.5707 0  0; parent link_chassis -> base_link
- joint joint_sensor_laser: parent link_chassis -> base_link
